File: imx_pequena/imx_mpu.kicad_sch (KiCad schematic)
At the start: 0 parts

Commit message: lots of updates
Set design rules, fixed ERC, etc....
Other:
- sheet pinouts ports: added I2C1_SCL, I2C1_SDA, I2C2_SCL, I2C2_SDA, UART1_CTS, UART1_RTS, UART1_RX, UART1_TX, UART2_CTS, UART2_RTS, UART2_RX, UART2_TX, UART3_RX, UART3_TX; removed none
Changed lines of the file:
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@@
+    (stroke (width 0) (type default) (color 0 0 0 0))
+  )
+  (wire (pts (xy 198.12 45.72) (xy 203.2 45.72))
     (stroke (width 0) (type default) (color 0 0 0 0))
   )
@@
     (stroke (width 0) (type default) (color 0 0 0 0))
   )
+  (wire (pts (xy 203.2 55.88) (xy 198.12 55.88))
+    (stroke (width 0) (type default) (color 0 0 0 0))
+  )
   (wire (pts (xy 71.12 48.26) (xy 72.39 48.26))
     (stroke (width 0) (type default) (color 0 0 0 0))
   )
+  (wire (pts (xy 203.2 81.28) (xy 198.12 81.28))
+    (stroke (width 0) (type default) (color 0 0 0 0))
+  )
   (wire (pts (xy 71.12 40.64) (xy 72.39 40.64))
     (stroke (width 0) (type default) (color 0 0 0 0))
   )
+  (wire (pts (xy 198.12 76.2) (xy 203.2 76.2))
+    (stroke (width 0) (type default) (color 0 0 0 0))
+  )
   (wire (pts (xy 101.6 76.2) (xy 106.68 76.2))
     (stroke (width 0) (type default) (color 0 0 0 0))
@@
     (stroke (width 0) (type default) (color 0 0 0 0))
   )
+  (wire (pts (xy 198.12 43.18) (xy 203.2 43.18))
+    (stroke (width 0) (type default) (color 0 0 0 0))
+  )
+  (wire (pts (xy 203.2 60.96) (xy 198.12 60.96))
+    (stroke (width 0) (type default) (color 0 0 0 0))
+  )
+  (wire (pts (xy 203.2 83.82) (xy 198.12 83.82))
+    (stroke (width 0) (type default) (color 0 0 0 0))
+  )
   (wire (pts (xy 147.32 81.28) (xy 152.4 81.28))
     (stroke (width 0) (type default) (color 0 0 0 0))
@@
     (stroke (width 0) (type default) (color 0 0 0 0))
   )
+  (wire (pts (xy 203.2 66.04) (xy 198.12 66.04))
+    (stroke (width 0) (type default) (color 0 0 0 0))
+  )
   (wire (pts (xy 71.12 45.72) (xy 72.39 45.72))
     (stroke (width 0) (type default) (color 0 0 0 0))
   )
+  (wire (pts (xy 198.12 73.66) (xy 203.2 73.66))
+    (stroke (width 0) (type default) (color 0 0 0 0))
+  )
+  (wire (pts (xy 203.2 58.42) (xy 198.12 58.42))
+    (stroke (width 0) (type default) (color 0 0 0 0))
+  )
   (wire (pts (xy 71.12 35.56) (xy 72.39 35.56))
     (stroke (width 0) (type default) (color 0 0 0 0))
@@
     (stroke (width 0) (type default) (color 0 0 0 0))
   )
+  (wire (pts (xy 198.12 40.64) (xy 203.2 40.64))
+    (stroke (width 0) (type default) (color 0 0 0 0))
+  )
+  (wire (pts (xy 203.2 53.34) (xy 198.12 53.34))
+    (stroke (width 0) (type default) (color 0 0 0 0))
+  )
+  (wire (pts (xy 198.12 38.1) (xy 203.2 38.1))
+    (stroke (width 0) (type default) (color 0 0 0 0))
+  )
   (wire (pts (xy 101.6 73.66) (xy 106.68 73.66))
     (stroke (width 0) (type default) (color 0 0 0 0))
@@
     (stroke (width 0) (type default) (color 0 0 0 0))
   )
+  (wire (pts (xy 203.2 68.58) (xy 198.12 68.58))
+    (stroke (width 0) (type default) (color 0 0 0 0))
+  )
   (wire (pts (xy 147.32 76.2) (xy 152.4 76.2))
     (stroke (width 0) (type default) (color 0 0 0 0))
@@
     (stroke (width 0) (type default) (color 0 0 0 0))
   )
+  (label "UART2_TX" (at 198.12 53.34 180)
+    (effects (font (size 1.27 1.27)) (justify right bottom))
+  )
   (label "UART3_RX" (at 152.4 93.98 0)
     (effects (font (size 1.27 1.27)) (justify left bottom))
   )
+  (label "I2C2_SDA" (at 198.12 83.82 180)
+    (effects (font (size 1.27 1.27)) (justify right bottom))
+  )
   (label "UART2_CTS" (at 152.4 81.28 0)
     (effects (font (size 1.27 1.27)) (justify left bottom))
   )
+  (label "UART2_RTS" (at 198.12 58.42 180)
+    (effects (font (size 1.27 1.27)) (justify right bottom))
+  )
   (label "UART1_RTS" (at 101.6 78.74 180)
     (effects (font (size 1.27 1.27)) (justify right bottom))
@@
     (effects (font (size 1.27 1.27)) (justify right bottom))
   )
+  (label "UART3_TX" (at 198.12 66.04 180)
+    (effects (font (size 1.27 1.27)) (justify right bottom))
+  )
   (label "UART2_TX" (at 152.4 73.66 0)
     (effects (font (size 1.27 1.27)) (justify left bottom))
   )
+  (label "UART1_RX" (at 198.12 40.64 180)
+    (effects (font (size 1.27 1.27)) (justify right bottom))
+  )
+  (label "UART3_RX" (at 198.12 68.58 180)
+    (effects (font (size 1.27 1.27)) (justify right bottom))
+  )
+  (label "UART1_TX" (at 198.12 38.1 180)
+    (effects (font (size 1.27 1.27)) (justify right bottom))
+  )
   (label "UART2_RTS" (at 152.4 78.74 0)
     (effects (font (size 1.27 1.27)) (justify left bottom))
   )
+  (label "UART1_CTS" (at 198.12 45.72 180)
+    (effects (font (size 1.27 1.27)) (justify right bottom))
+  )
   (label "I2C2_SDA" (at 76.2 57.15 0)
     (effects (font (size 1.27 1.27)) (justify left bottom))
   )
+  (label "UART1_RTS" (at 198.12 43.18 180)
+    (effects (font (size 1.27 1.27)) (justify right bottom))
+  )
+  (label "UART2_CTS" (at 198.12 60.96 180)
+    (effects (font (size 1.27 1.27)) (justify right bottom))
+  )
   (label "I2C1_SCL" (at 101.6 88.9 180)
     (effects (font (size 1.27 1.27)) (justify right bottom))
   )
+  (label "I2C2_SCL" (at 198.12 81.28 180)
+    (effects (font (size 1.27 1.27)) (justify right bottom))
+  )
   (label "UART3_TX" (at 152.4 91.44 0)
     (effects (font (size 1.27 1.27)) (justify left bottom))
   )
+  (label "I2C1_SDA" (at 198.12 76.2 180)
+    (effects (font (size 1.27 1.27)) (justify right bottom))
+  )
+  (label "UART2_RX" (at 198.12 55.88 180)
+    (effects (font (size 1.27 1.27)) (justify right bottom))
+  )
   (label "UART1_CTS" (at 101.6 81.28 180)
     (effects (font (size 1.27 1.27)) (justify right bottom))
@@
   (label "I2C2_SCL" (at 76.2 54.61 0)
     (effects (font (size 1.27 1.27)) (justify left bottom))
+  )
+  (label "I2C1_SCL" (at 198.12 73.66 180)
+    (effects (font (size 1.27 1.27)) (justify right bottom))
   )
   (hierarchical_label "USB1_DN" (shape bidirectional) (at 72.39 38.1 0)
@@
       (effects (font (size 1.27 1.27)) (justify left top))
     )
-  )
+    (pin "I2C2_SCL" input (at 203.2 81.28 180)
+      (effects (font (size 1.27 1.27)) (justify left))
+    )
+    (pin "I2C2_SDA" input (at 203.2 83.82 180)
+      (effects (font (size 1.27 1.27)) (justify left))
+    )
+    (pin "I2C1_SCL" input (at 203.2 73.66 180)
+      (effects (font (size 1.27 1.27)) (justify left))
+    )
+    (pin "I2C1_SDA" input (at 203.2 76.2 180)
+      (effects (font (size 1.27 1.27)) (justify left))
+    )
+    (pin "UART3_RX" input (at 203.2 68.58 180)
+      (effects (font (size 1.27 1.27)) (justify left))
+    )
+    (pin "UART1_RX" input (at 203.2 40.64 180)
+      (effects (font (size 1.27 1.27)) (justify left))
+    )
+    (pin "UART1_TX" input (at 203.2 38.1 180)
+      (effects (font (size 1.27 1.27)) (justify left))
+    )
+    (pin "UART2_CTS" input (at 203.2 60.96 180)
+      (effects (font (size 1.27 1.27)) (justify left))
+    )
+    (pin "UART2_TX" input (at 203.2 53.34 180)
+      (effects (font (size 1.27 1.27)) (justify left))
+    )
+    (pin "UART2_RX" input (at 203.2 55.88 180)
+      (effects (font (size 1.27 1.27)) (justify left))
+    )
+    (pin "UART2_RTS" input (at 203.2 58.42 180)
+      (effects (font (size 1.27 1.27)) (justify left))
+    )
+    (pin "UART3_TX" input (at 203.2 66.04 180)
+      (effects (font (size 1.27 1.27)) (justify left))
+    )
+    (pin "UART1_RTS" input (at 203.2 43.18 180)
+      (effects (font (size 1.27 1.27)) (justify left))
+    )
+    (pin "UART1_CTS" input (at 203.2 45.72 180)
+      (effects (font (size 1.27 1.27)) (justify left))
+    )
+  )
