File: imx_pequena/imx_usb.kicad_sch (KiCad schematic)
At the start: 12 parts

Commit message: Power Update
Added 3v3 and 1.35V switchers
Parts:
- gave numbers to parts that had none: 12
Changed lines of the file:
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@@
   (symbol (lib_id "power:GND") (at 44.45 128.27 0) (unit 1)
     (in_bom yes) (on_board yes) (fields_autoplaced)
-    (property "Reference" "#PWR?" (id 0) (at 44.45 134.62 0)
+    (property "Reference" "#PWR0128" (id 0) (at 44.45 134.62 0)
       (effects (font (size 1.27 1.27)) hide)
     )
@@
   (symbol (lib_id "power:GND") (at 64.77 52.07 0) (unit 1)
     (in_bom yes) (on_board yes) (fields_autoplaced)
-    (property "Reference" "#PWR?" (id 0) (at 64.77 58.42 0)
+    (property "Reference" "#PWR0126" (id 0) (at 64.77 58.42 0)
       (effects (font (size 1.27 1.27)) hide)
     )
@@
   (symbol (lib_id "Device:R_Small_US") (at 38.1 119.38 90) (unit 1)
     (in_bom yes) (on_board yes)
-    (property "Reference" "R?" (id 0) (at 35.56 118.11 90))
+    (property "Reference" "R16" (id 0) (at 35.56 118.11 90))
     (property "Value" "22" (id 1) (at 38.1 121.92 90))
     (property "Footprint" "" (id 2) (at 38.1 119.38 0)
@@
   (symbol (lib_id "Device:C_Small") (at 44.45 124.46 0) (unit 1)
     (in_bom yes) (on_board yes)
-    (property "Reference" "C?" (id 0) (at 45.72 123.19 0)
+    (property "Reference" "C41" (id 0) (at 45.72 123.19 0)
       (effects (font (size 1.27 1.27)) (justify left))
     )
@@
   (symbol (lib_id "Device:C_Small") (at 50.8 124.46 0) (unit 1)
     (in_bom yes) (on_board yes)
-    (property "Reference" "C?" (id 0) (at 52.07 123.19 0)
+    (property "Reference" "C42" (id 0) (at 52.07 123.19 0)
       (effects (font (size 1.27 1.27)) (justify left))
     )
@@
   (symbol (lib_id "Device:C_Small") (at 64.77 48.26 0) (unit 1)
     (in_bom yes) (on_board yes)
-    (property "Reference" "C?" (id 0) (at 66.04 46.99 0)
+    (property "Reference" "C43" (id 0) (at 66.04 46.99 0)
       (effects (font (size 1.27 1.27)) (justify left))
     )
@@
   (symbol (lib_id "power:GND") (at 29.21 93.98 0) (unit 1)
     (in_bom yes) (on_board yes) (fields_autoplaced)
-    (property "Reference" "#PWR?" (id 0) (at 29.21 100.33 0)
+    (property "Reference" "#PWR0125" (id 0) (at 29.21 100.33 0)
       (effects (font (size 1.27 1.27)) hide)
     )
@@
   (symbol (lib_id "Device:R_Small_US") (at 48.26 33.02 90) (unit 1)
     (in_bom yes) (on_board yes)
-    (property "Reference" "R?" (id 0) (at 44.45 34.29 90))
+    (property "Reference" "R18" (id 0) (at 44.45 34.29 90))
     (property "Value" "5.1K" (id 1) (at 48.26 35.56 90))
     (property "Footprint" "" (id 2) (at 48.26 33.02 0)
@@
   (symbol (lib_id "power:GND") (at 50.8 128.27 0) (unit 1)
     (in_bom yes) (on_board yes) (fields_autoplaced)
-    (property "Reference" "#PWR?" (id 0) (at 50.8 134.62 0)
+    (property "Reference" "#PWR0129" (id 0) (at 50.8 134.62 0)
       (effects (font (size 1.27 1.27)) hide)
     )
@@
   (symbol (lib_id "power:GND") (at 21.59 93.98 0) (unit 1)
     (in_bom yes) (on_board yes) (fields_autoplaced)
-    (property "Reference" "#PWR?" (id 0) (at 21.59 100.33 0)
+    (property "Reference" "#PWR0127" (id 0) (at 21.59 100.33 0)
       (effects (font (size 1.27 1.27)) hide)
     )
@@
   (symbol (lib_id "Device:R_Small_US") (at 59.69 39.37 90) (unit 1)
     (in_bom yes) (on_board yes)
-    (property "Reference" "R?" (id 0) (at 57.15 38.1 90))
+    (property "Reference" "R19" (id 0) (at 57.15 38.1 90))
     (property "Value" "22" (id 1) (at 59.69 36.83 90))
     (property "Footprint" "" (id 2) (at 59.69 39.37 0)
@@
   (symbol (lib_id "power:GND") (at 52.07 34.29 0) (unit 1)
     (in_bom yes) (on_board yes)
-    (property "Reference" "#PWR?" (id 0) (at 52.07 40.64 0)
+    (property "Reference" "#PWR0123" (id 0) (at 52.07 40.64 0)
       (effects (font (size 1.27 1.27)) hide)
     )
@@
   (symbol (lib_id "power:GND") (at 22.86 129.54 0) (unit 1)
     (in_bom yes) (on_board yes) (fields_autoplaced)
-    (property "Reference" "#PWR?" (id 0) (at 22.86 135.89 0)
+    (property "Reference" "#PWR0130" (id 0) (at 22.86 135.89 0)
       (effects (font (size 1.27 1.27)) hide)
     )
@@
   (symbol (lib_id "Device:R_Small_US") (at 48.26 30.48 90) (unit 1)
     (in_bom yes) (on_board yes)
-    (property "Reference" "R?" (id 0) (at 45.72 29.21 90))
+    (property "Reference" "R17" (id 0) (at 45.72 29.21 90))
     (property "Value" "5.1K" (id 1) (at 52.07 29.21 90))
     (property "Footprint" "" (id 2) (at 48.26 30.48 0)
@@
   (symbol (lib_id "Connector:USB_C_Receptacle") (at 29.21 50.8 0) (unit 1)
     (in_bom yes) (on_board yes) (fields_autoplaced)
-    (property "Reference" "J?" (id 0) (at 29.21 17.78 0))
+    (property "Reference" "J4" (id 0) (at 29.21 17.78 0))
     (property "Value" "USB_C_Receptacle" (id 1) (at 29.21 20.32 0))
     (property "Footprint" "" (id 2) (at 33.02 50.8 0)
@@
   (symbol (lib_id "Device:C_Small") (at 71.12 48.26 0) (unit 1)
     (in_bom yes) (on_board yes)
-    (property "Reference" "C?" (id 0) (at 72.39 46.99 0)
+    (property "Reference" "C44" (id 0) (at 72.39 46.99 0)
       (effects (font (size 1.27 1.27)) (justify left))
     )
@@
   (symbol (lib_id "Device:R_Small_US") (at 59.69 44.45 90) (unit 1)
     (in_bom yes) (on_board yes)
-    (property "Reference" "R?" (id 0) (at 57.15 43.18 90))
+    (property "Reference" "R20" (id 0) (at 57.15 43.18 90))
     (property "Value" "22" (id 1) (at 59.69 46.99 90))
     (property "Footprint" "" (id 2) (at 59.69 44.45 0)
@@
   (symbol (lib_id "Connector:USB_B_Micro") (at 24.13 116.84 0) (unit 1)
     (in_bom yes) (on_board yes) (fields_autoplaced)
-    (property "Reference" "J?" (id 0) (at 24.13 104.14 0))
+    (property "Reference" "J3" (id 0) (at 24.13 104.14 0))
     (property "Value" "USB_B_Micro" (id 1) (at 24.13 106.68 0))
     (property "Footprint" "" (id 2) (at 27.94 118.11 0)
@@
   (symbol (lib_id "Device:R_Small_US") (at 38.1 116.84 90) (unit 1)
     (in_bom yes) (on_board yes)
-    (property "Reference" "R?" (id 0) (at 35.56 115.57 90))
+    (property "Reference" "R15" (id 0) (at 35.56 115.57 90))
     (property "Value" "22" (id 1) (at 38.1 114.3 90))
     (property "Footprint" "" (id 2) (at 38.1 116.84 0)
@@
   (symbol (lib_id "power:GND") (at 71.12 52.07 0) (unit 1)
     (in_bom yes) (on_board yes) (fields_autoplaced)
-    (property "Reference" "#PWR?" (id 0) (at 71.12 58.42 0)
-      (effects (font (size 1.27 1.27)) hide)
-    )
+    (property "Reference" "#PWR0124" (id 0) (at 71.12 58.42 0)
+      (effects (font (size 1.27 1.27)) hide)
+    )

Commit message: Cleaned up NVCC pins
Added 3v3 connections + decoupling caps to NVcc pins
Parts:
- added D?: D_TVS, symbol Device:D_TVS
- added F? (x2): Fuse_Small, symbol Device:Fuse_Small
Connections:
- net GND: now also D?.1 (A1)
- net USB1_VBUS: now also F?.2; no longer J3.1 (VBUS)
- net USB2_VBUS: now also D?.2 (A2), F?.2; no longer J4.A4 (VBUS), J4.A9 (VBUS), J4.B4 (VBUS), J4.B9 (VBUS)
- new net: F?.1, J3.1 (VBUS)
- new net: F?.1, J4.A4 (VBUS), J4.A9 (VBUS), J4.B4 (VBUS), J4.B9 (VBUS)
Changed lines of the file:
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@@
   (junction (at 52.07 33.02) (diameter 0) (color 0 0 0 0)
   )
+  (junction (at 72.39 25.4) (diameter 0) (color 0 0 0 0)
+  )
   (wire (pts (xy 62.23 44.45) (xy 64.77 44.45))
     (stroke (width 0) (type default) (color 0 0 0 0))
@@
     (stroke (width 0) (type default) (color 0 0 0 0))
   )
+  (wire (pts (xy 72.39 25.4) (xy 90.17 25.4))
+    (stroke (width 0) (type default) (color 0 0 0 0))
+  )
+  (wire (pts (xy 72.39 34.29) (xy 72.39 35.56))
+    (stroke (width 0) (type default) (color 0 0 0 0))
+  )
   (wire (pts (xy 44.45 119.38) (xy 44.45 121.92))
     (stroke (width 0) (type default) (color 0 0 0 0))
@@
     (stroke (width 0) (type default) (color 0 0 0 0))
   )
+  (wire (pts (xy 40.64 111.76) (xy 57.15 111.76))
+    (stroke (width 0) (type default) (color 0 0 0 0))
+  )
+  (wire (pts (xy 58.42 25.4) (xy 72.39 25.4))
+    (stroke (width 0) (type default) (color 0 0 0 0))
+  )
   (wire (pts (xy 50.8 30.48) (xy 52.07 30.48))
     (stroke (width 0) (type default) (color 0 0 0 0))
@@
     (stroke (width 0) (type default) (color 0 0 0 0))
   )
-  (wire (pts (xy 44.45 25.4) (xy 45.72 25.4))
-    (stroke (width 0) (type default) (color 0 0 0 0))
-  )
   (wire (pts (xy 52.07 30.48) (xy 52.07 33.02))
     (stroke (width 0) (type default) (color 0 0 0 0))
@@
     (stroke (width 0) (type default) (color 0 0 0 0))
   )
+  (wire (pts (xy 44.45 25.4) (xy 53.34 25.4))
+    (stroke (width 0) (type default) (color 0 0 0 0))
+  )
   (wire (pts (xy 24.13 127) (xy 24.13 129.54))
     (stroke (width 0) (type default) (color 0 0 0 0))
@@
     (stroke (width 0) (type default) (color 0 0 0 0))
   )
-  (wire (pts (xy 31.75 111.76) (xy 33.02 111.76))
+  (wire (pts (xy 31.75 111.76) (xy 35.56 111.76))
     (stroke (width 0) (type default) (color 0 0 0 0))
   )
@@
     (stroke (width 0) (type default) (color 0 0 0 0))
   )
+  (wire (pts (xy 72.39 25.4) (xy 72.39 26.67))
+    (stroke (width 0) (type default) (color 0 0 0 0))
+  )
   (wire (pts (xy 40.64 119.38) (xy 44.45 119.38))
     (stroke (width 0) (type default) (color 0 0 0 0))
@@
     (effects (font (size 1.27 1.27)) (justify left))
   )
-  (hierarchical_label "USB2_VBUS" (shape bidirectional) (at 45.72 25.4 0)
-    (effects (font (size 1.27 1.27)) (justify left))
-  )
-  (hierarchical_label "USB1_VBUS" (shape bidirectional) (at 33.02 111.76 0)
+  (hierarchical_label "USB2_VBUS" (shape bidirectional) (at 90.17 25.4 0)
+    (effects (font (size 1.27 1.27)) (justify left))
+  )
+  (hierarchical_label "USB1_VBUS" (shape bidirectional) (at 57.15 111.76 0)
     (effects (font (size 1.27 1.27)) (justify left))
   )
@@
     )
     (pin "1")
+  )
+  (symbol (lib_id "power:GND") (at 72.39 35.56 0) (unit 1)
+    (in_bom yes) (on_board yes)
+    (property "Reference" "#PWR?" (id 0) (at 72.39 41.91 0)
+      (effects (font (size 1.27 1.27)) hide)
+    )
+    (property "Value" "GND" (id 1) (at 74.93 35.56 0))
+    (property "Footprint" "" (id 2) (at 72.39 35.56 0)
+      (effects (font (size 1.27 1.27)) hide)
+    )
+    (property "Datasheet" "" (id 3) (at 72.39 35.56 0)
+      (effects (font (size 1.27 1.27)) hide)
+    )
+    (pin "1")
+  )
+  (symbol (lib_id "Device:Fuse_Small") (at 38.1 111.76 0) (unit 1)
+    (in_bom yes) (on_board yes) (fields_autoplaced)
+    (property "Reference" "F?" (id 0) (at 38.1 106.68 0))
+    (property "Value" "Fuse_Small" (id 1) (at 38.1 109.22 0))
+    (property "Footprint" "" (id 2) (at 38.1 111.76 0)
+      (effects (font (size 1.27 1.27)) hide)
+    )
+    (property "Datasheet" "~" (id 3) (at 38.1 111.76 0)
+      (effects (font (size 1.27 1.27)) hide)
+    )
+    (pin "1")
+    (pin "2")
   )
   (symbol (lib_id "power:GND") (at 64.77 52.07 0) (unit 1)
@@
     )
     (property "Datasheet" "~" (id 3) (at 48.26 33.02 0)
+      (effects (font (size 1.27 1.27)) hide)
+    )
+    (pin "1")
+    (pin "2")
+  )
+  (symbol (lib_id "Device:Fuse_Small") (at 55.88 25.4 0) (unit 1)
+    (in_bom yes) (on_board yes) (fields_autoplaced)
+    (property "Reference" "F?" (id 0) (at 55.88 20.32 0))
+    (property "Value" "Fuse_Small" (id 1) (at 55.88 22.86 0))
+    (property "Footprint" "" (id 2) (at 55.88 25.4 0)
+      (effects (font (size 1.27 1.27)) hide)
+    )
+    (property "Datasheet" "~" (id 3) (at 55.88 25.4 0)
       (effects (font (size 1.27 1.27)) hide)
     )
@@
     (pin "6")
   )
+  (symbol (lib_id "Device:D_TVS") (at 72.39 30.48 90) (unit 1)
+    (in_bom yes) (on_board yes) (fields_autoplaced)
+    (property "Reference" "D?" (id 0) (at 74.93 29.2099 90)
+      (effects (font (size 1.27 1.27)) (justify right))
+    )
+    (property "Value" "D_TVS" (id 1) (at 74.93 31.7499 90)
+      (effects (font (size 1.27 1.27)) (justify right))
+    )
+    (property "Footprint" "" (id 2) (at 72.39 30.48 0)
+      (effects (font (size 1.27 1.27)) hide)
+    )
+    (property "Datasheet" "~" (id 3) (at 72.39 30.48 0)
+      (effects (font (size 1.27 1.27)) hide)
+    )
+    (pin "1")
+    (pin "2")
+  )
   (symbol (lib_id "Device:R_Small_US") (at 38.1 116.84 90) (unit 1)
