File: imx_pequena/mpu_d_uart.kicad_sch (KiCad schematic)
At the start: 7 parts, among them J3 Conn_01x04, U1 MCIMX6Z0DVM09AB

Commit message: lots of updates
Set design rules, fixed ERC, etc....
Connections:
- no-connect marks 0 -> 2
Changed lines of the file:
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@@
   (junction (at 68.58 96.52) (diameter 0) (color 0 0 0 0)
   )
+  (no_connect (at 93.98 86.36))
+  (no_connect (at 93.98 83.82))
   (wire (pts (xy 175.26 62.23) (xy 179.07 62.23))
     (stroke (width 0) (type default) (color 0 0 0 0))
@@
   )
   (wire (pts (xy 185.42 53.34) (xy 189.23 53.34))
+    (stroke (width 0) (type default) (color 0 0 0 0))
+  )
+  (wire (pts (xy 93.98 83.82) (xy 102.87 83.82))
     (stroke (width 0) (type default) (color 0 0 0 0))
   )
@@
     (stroke (width 0) (type default) (color 0 0 0 0))
   )
+  (wire (pts (xy 93.98 86.36) (xy 102.87 86.36))
+    (stroke (width 0) (type default) (color 0 0 0 0))
+  )
