File: imx_pequena/pinouts.kicad_sch (KiCad schematic)
At the start: 0 parts

Commit message: Part Assignment
Assigned GPIOs and assigned footprints to most parts
Parts:
- added J10, J11, J12, J6, J7, J8, J9: Conn_02x06_Top_Bottom, Connector_PinHeader_2.54mm:PinHeader_2x06_P2.54mm_Horizontal, symbol Connector_Generic:Conn_02x06_Top_Bottom
Connections:
- new net 3v3: J10.12 (Pin_12), J10.6 (Pin_6), J11.12 (Pin_12), J11.6 (Pin_6), J12.12 (Pin_12), J12.6 (Pin_6), J6.12 (Pin_12), J6.6 (Pin_6), J7.12 (Pin_12), J7.6 (Pin_6), J8.12 (Pin_12), J8.6 (Pin_6), J9.12 (Pin_12), J9.6 (Pin_6)
- new net GND: J10.11 (Pin_11), J10.5 (Pin_5), J11.11 (Pin_11), J11.5 (Pin_5), J12.11 (Pin_11), J12.5 (Pin_5), J6.11 (Pin_11), J6.5 (Pin_5), J7.11 (Pin_11), J7.5 (Pin_5), J8.11 (Pin_11), J8.5 (Pin_5), J9.11 (Pin_11), J9.5 (Pin_5)
- new net GPIO1_0: J9.7 (Pin_7)
- new net GPIO1_1: J9.8 (Pin_8)
- new net GPIO1_2: J9.9 (Pin_9)
- new net GPIO1_3: J9.10 (Pin_10)
- new net GPIO1_4: J11.7 (Pin_7)
- new net GPIO1_6: J11.8 (Pin_8)
- new net GPIO1_7: J11.9 (Pin_9)
- new net GPIO3_0: J7.7 (Pin_7)
- new net GPIO3_1: J7.8 (Pin_8)
- new net GPIO3_13: J10.7 (Pin_7)
- new net GPIO3_14: J10.8 (Pin_8)
- new net GPIO3_15: J10.9 (Pin_9)
- new net GPIO3_16: J10.10 (Pin_10)
- new net GPIO3_18: J8.1 (Pin_1)
- new net GPIO3_19: J8.3 (Pin_3)
- new net GPIO3_2: J7.9 (Pin_9)
- new net GPIO3_20: J8.4 (Pin_4)
- new net GPIO3_21: J8.7 (Pin_7)
- new net GPIO3_22: J8.10 (Pin_10)
- new net GPIO3_23: J8.9 (Pin_9)
- new net GPIO3_24: J11.10 (Pin_10)
- new net GPIO3_3: J7.10 (Pin_10)
- new net GPIO3_4: J12.1 (Pin_1)
- new net GPIO3_5: J12.3 (Pin_3)
- new net GPIO3_6: J12.4 (Pin_4)
- new net GPIO3_8: J12.7 (Pin_7)
- new net GPIO3_9: J12.9 (Pin_9)
- new net I2C1_SCL: J9.3 (Pin_3)
- new net I2C1_SDA: J9.4 (Pin_4)
- new net I2C2_SCL: J11.3 (Pin_3)
- new net I2C2_SDA: J11.4 (Pin_4)
- new net PWM1_out: J12.2 (Pin_2)
- new net PWM2_out: J12.8 (Pin_8)
- new net PWM3_out: J8.2 (Pin_2)
- new net PWM4_out: J8.8 (Pin_8)
- new net UART1_CTS: J10.1 (Pin_1)
- new net UART1_RTS: J10.4 (Pin_4)
- new net UART1_RX: J10.3 (Pin_3)
- new net UART1_TX: J10.2 (Pin_2)
- new net UART2_CTS: J7.1 (Pin_1)
- new net UART2_RTS: J7.4 (Pin_4)
- new net UART2_RX: J7.3 (Pin_3)
- new net UART2_TX: J7.2 (Pin_2)
- new net ecspi_miso: J6.3 (Pin_3)
- new net ecspi_mosi: J6.2 (Pin_2)
- new net ecspi_rdy: J6.7 (Pin_7)
- new net ecspi_sclk: J6.4 (Pin_4)
- new net ecspi_ss0: J6.1 (Pin_1)
- new net ecspi_ss1: J6.8 (Pin_8)
- new net ecspi_ss2: J6.9 (Pin_9)
- new net ecspi_ss3: J6.10 (Pin_10)

Commit message: lots of updates
Set design rules, fixed ERC, etc....
Connections:
- net UART3_RX: now also J11.2 (Pin_2)
- net UART3_TX: now also J11.1 (Pin_1)
- no-connect marks 0 -> 3
Changed lines of the file:
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@@
 (kicad_sch (version 20211123) (generator eeschema)
   (paper "A4")
+  (no_connect (at 88.9 49.53))
+  (no_connect (at 163.83 85.09))
+  (no_connect (at 88.9 52.07))
   (wire (pts (xy 41.91 59.69) (xy 50.8 59.69))
     (stroke (width 0) (type default) (color 0 0 0 0))
@@
     (stroke (width 0) (type default) (color 0 0 0 0))
   )
+  (wire (pts (xy 88.9 52.07) (xy 97.79 52.07))
+    (stroke (width 0) (type default) (color 0 0 0 0))
+  )
   (wire (pts (xy 63.5 116.84) (xy 64.77 116.84))
     (stroke (width 0) (type default) (color 0 0 0 0))
@@
     (stroke (width 0) (type default) (color 0 0 0 0))
   )
+  (wire (pts (xy 88.9 49.53) (xy 97.79 49.53))
+    (stroke (width 0) (type default) (color 0 0 0 0))
+  )
   (wire (pts (xy 35.56 186.69) (xy 30.48 186.69))
     (stroke (width 0) (type default) (color 0 0 0 0))
@@
     (stroke (width 0) (type default) (color 0 0 0 0))
   )
+  (wire (pts (xy 137.16 49.53) (xy 142.24 49.53))
+    (stroke (width 0) (type default) (color 0 0 0 0))
+  )
   (wire (pts (xy 35.56 161.29) (xy 30.48 161.29))
     (stroke (width 0) (type default) (color 0 0 0 0))
   )
+  (wire (pts (xy 137.16 52.07) (xy 142.24 52.07))
+    (stroke (width 0) (type default) (color 0 0 0 0))
+  )
   (wire (pts (xy 41.91 87.63) (xy 50.8 87.63))
     (stroke (width 0) (type default) (color 0 0 0 0))
@@
     (stroke (width 0) (type default) (color 0 0 0 0))
   )
+  (wire (pts (xy 154.94 85.09) (xy 163.83 85.09))
+    (stroke (width 0) (type default) (color 0 0 0 0))
+  )
   (wire (pts (xy 110.49 82.55) (xy 111.76 82.55))
     (stroke (width 0) (type default) (color 0 0 0 0))
@@
     (effects (font (size 1.27 1.27)) (justify right bottom))
   )
+  (label "UART3_TX" (at 137.16 49.53 180)
+    (effects (font (size 1.27 1.27)) (justify right bottom))
+  )
   (label "UART1_TX" (at 90.17 80.01 180)
     (effects (font (size 1.27 1.27)) (justify right bottom))
@@
     (effects (font (size 1.27 1.27)) (justify left bottom))
   )
+  (label "UART3_RX" (at 137.16 52.07 180)
+    (effects (font (size 1.27 1.27)) (justify right bottom))
+  )
   (label "UART2_RTS" (at 35.56 151.13 0)

Commit message: fixed part alllocation
fixed socket to pin header issue
Parts:
- J10, J11, J12, J6, J7, J8, J9: footprint Connector_PinHeader_2.54mm:PinHeader_2x06_P2.54mm_Horizontal -> Connector_PinSocket_2.54mm:PinSocket_2x06_P2.54mm_Horizontal
Changed lines of the file:
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@@
     (property "Reference" "J8" (id 0) (at 57.15 97.79 0))
     (property "Value" "Conn_02x06_Top_Bottom" (id 1) (at 57.15 100.33 0))
-    (property "Footprint" "Connector_PinHeader_2.54mm:PinHeader_2x06_P2.54mm_Horizontal" (id 2) (at 55.88 109.22 0)
+    (property "Footprint" "Connector_PinSocket_2.54mm:PinSocket_2x06_P2.54mm_Horizontal" (id 2) (at 55.88 109.22 0)
       (effects (font (size 1.27 1.27)) hide)
     )
@@
     (property "Reference" "J11" (id 0) (at 148.59 43.18 0))
     (property "Value" "Conn_02x06_Top_Bottom" (id 1) (at 148.59 45.72 0))
-    (property "Footprint" "Connector_PinHeader_2.54mm:PinHeader_2x06_P2.54mm_Horizontal" (id 2) (at 147.32 54.61 0)
+    (property "Footprint" "Connector_PinSocket_2.54mm:PinSocket_2x06_P2.54mm_Horizontal" (id 2) (at 147.32 54.61 0)
       (effects (font (size 1.27 1.27)) hide)
     )
@@
     (property "Reference" "J12" (id 0) (at 148.59 71.12 0))
     (property "Value" "Conn_02x06_Top_Bottom" (id 1) (at 148.59 73.66 0))
-    (property "Footprint" "Connector_PinHeader_2.54mm:PinHeader_2x06_P2.54mm_Horizontal" (id 2) (at 147.32 82.55 0)
+    (property "Footprint" "Connector_PinSocket_2.54mm:PinSocket_2x06_P2.54mm_Horizontal" (id 2) (at 147.32 82.55 0)
       (effects (font (size 1.27 1.27)) hide)
     )
@@
     (property "Reference" "J9" (id 0) (at 104.14 43.18 0))
     (property "Value" "Conn_02x06_Top_Bottom" (id 1) (at 104.14 45.72 0))
-    (property "Footprint" "Connector_PinHeader_2.54mm:PinHeader_2x06_P2.54mm_Horizontal" (id 2) (at 102.87 54.61 0)
+    (property "Footprint" "Connector_PinSocket_2.54mm:PinSocket_2x06_P2.54mm_Horizontal" (id 2) (at 102.87 54.61 0)
       (effects (font (size 1.27 1.27)) hide)
     )
@@
     (property "Reference" "J6" (id 0) (at 57.15 43.18 0))
     (property "Value" "Conn_02x06_Top_Bottom" (id 1) (at 57.15 45.72 0))
-    (property "Footprint" "Connector_PinHeader_2.54mm:PinHeader_2x06_P2.54mm_Horizontal" (id 2) (at 55.88 54.61 0)
+    (property "Footprint" "Connector_PinSocket_2.54mm:PinSocket_2x06_P2.54mm_Horizontal" (id 2) (at 55.88 54.61 0)
       (effects (font (size 1.27 1.27)) hide)
     )
@@
     (property "Reference" "J7" (id 0) (at 57.15 71.12 0))
     (property "Value" "Conn_02x06_Top_Bottom" (id 1) (at 57.15 73.66 0))
-    (property "Footprint" "Connector_PinHeader_2.54mm:PinHeader_2x06_P2.54mm_Horizontal" (id 2) (at 55.88 82.55 0)
+    (property "Footprint" "Connector_PinSocket_2.54mm:PinSocket_2x06_P2.54mm_Horizontal" (id 2) (at 55.88 82.55 0)
       (effects (font (size 1.27 1.27)) hide)
     )
@@
     (property "Reference" "J10" (id 0) (at 104.14 71.12 0))
     (property "Value" "Conn_02x06_Top_Bottom" (id 1) (at 104.14 73.66 0))
-    (property "Footprint" "Connector_PinHeader_2.54mm:PinHeader_2x06_P2.54mm_Horizontal" (id 2) (at 102.87 82.55 0)
-      (effects (font (size 1.27 1.27)) hide)
-    )
+    (property "Footprint" "Connector_PinSocket_2.54mm:PinSocket_2x06_P2.54mm_Horizontal" (id 2) (at 102.87 82.55 0)
+      (effects (font (size 1.27 1.27)) hide)
+    )
